File: sch/ram.kicad_sch (KiCad schematic)
At the start: 26 parts

Commit message: Schematics completed with values
Visual corrections pending
Parts:
- D20, D21, D22, D23, D24, D25, D26: CCCP (none) -> КР565РУ5Д
- D51, D52, D53, D54: value 74LS153 -> 74153
Changed lines of the file:
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@@
+      (effects (font (size 1.27 1.27)) hide)
+    )
+    (property "CCCP" "КР565РУ5Д" (id 4) (at 137.16 31.75 0)
       (effects (font (size 1.27 1.27)) hide)
     )
@@
       (effects (font (size 1.27 1.27)) hide)
     )
+    (property "CCCP" "КР565РУ5Д" (id 4) (at 210.82 31.75 0)
+      (effects (font (size 1.27 1.27)) hide)
+    )
     (pin "")
     (pin "10")
@@
       (effects (font (size 1.27 1.27)) (justify left))
     )
-    (property "Value" "74LS153" (id 1) (at 155.6894 134.62 0)
+    (property "Value" "74153" (id 1) (at 155.6894 134.62 0)
       (effects (font (size 1.27 1.27)) (justify left))
     )
@@
       (effects (font (size 1.27 1.27)) (justify left))
     )
-    (property "Value" "74LS153" (id 1) (at 87.1094 134.62 0)
+    (property "Value" "74153" (id 1) (at 87.1094 134.62 0)
       (effects (font (size 1.27 1.27)) (justify left))
     )
@@
       (effects (font (size 1.27 1.27)) hide)
     )
+    (property "CCCP" "КР565РУ5Д" (id 4) (at 247.65 31.75 0)
+      (effects (font (size 1.27 1.27)) hide)
+    )
     (pin "")
     (pin "10")
@@
       (effects (font (size 1.27 1.27)) (justify left))
     )
-    (property "Value" "74LS153" (id 1) (at 224.2694 134.62 0)
+    (property "Value" "74153" (id 1) (at 224.2694 134.62 0)
       (effects (font (size 1.27 1.27)) (justify left))
     )
@@
       (effects (font (size 1.27 1.27)) hide)
     )
+    (property "CCCP" "КР565РУ5Д" (id 4) (at 173.99 31.75 0)
+      (effects (font (size 1.27 1.27)) hide)
+    )
     (pin "")
     (pin "10")
@@
       (effects (font (size 1.27 1.27)) hide)
     )
+    (property "CCCP" "КР565РУ5Д" (id 4) (at 100.33 31.75 0)
+      (effects (font (size 1.27 1.27)) hide)
+    )
     (pin "")
     (pin "10")
@@
       (effects (font (size 1.27 1.27)) hide)
     )
+    (property "CCCP" "КР565РУ5Д" (id 4) (at 321.31 31.75 0)
+      (effects (font (size 1.27 1.27)) hide)
+    )
     (pin "")
     (pin "10")
@@
       (effects (font (size 1.27 1.27)) (justify left))
     )
-    (property "Value" "74LS153" (id 1) (at 292.8494 134.62 0)
+    (property "Value" "74153" (id 1) (at 292.8494 134.62 0)
       (effects (font (size 1.27 1.27)) (justify left))
     )
@@
       (effects (font (size 1.27 1.27)) hide)
     )
+    (property "CCCP" "КР565РУ5Д" (id 4) (at 284.48 31.75 0)
+      (effects (font (size 1.27 1.27)) hide)
+    )
