File: sch/video.kicad_sch (KiCad schematic)
At the start: 28 parts, among them X5 DIN-7

Commit message: Sch: visual corrections
Parts:
- C57: value (none) -> 200pF
- X5: value DIN-7 -> Video
Changed lines of the file:
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@@
   )
   (symbol (lib_id "Device:R_Small") (at 330.962 64.77 90) (unit 1)
-    (in_bom yes) (on_board yes) (fields_autoplaced)
+    (in_bom yes) (on_board yes)
     (property "Reference" "R25" (id 0) (at 330.962 58.42 90))
     (property "Value" "150R" (id 1) (at 330.962 60.96 90))
@@
       (effects (font (size 1.27 1.27)) (justify left))
     )
-    (property "Value" "" (id 1) (at 93.98 94.6212 0)
+    (property "Value" "200pF" (id 1) (at 93.98 94.6212 0)
       (effects (font (size 1.27 1.27)) (justify left))
     )
@@
   )
   (symbol (lib_id "Device:C_Polarized_Small") (at 324.485 64.77 90) (unit 1)
-    (in_bom yes) (on_board yes) (fields_autoplaced)
-    (property "Reference" "C54" (id 0) (at 323.9389 58.42 90))
-    (property "Value" "50μF/6.3V" (id 1) (at 323.9389 60.96 90))
+    (in_bom yes) (on_board yes)
+    (property "Reference" "C54" (id 0) (at 324.485 61.595 90))
+    (property "Value" "50μF/6.3V" (id 1) (at 324.485 67.945 90))
     (property "Footprint" "" (id 2) (at 324.485 64.77 0)
       (effects (font (size 1.27 1.27)) hide)
@@
   )
   (symbol (lib_id "Device:C_Polarized_Small") (at 324.485 81.28 90) (unit 1)
-    (in_bom yes) (on_board yes) (fields_autoplaced)
-    (property "Reference" "C53" (id 0) (at 323.9389 74.93 90))
-    (property "Value" "50μF/6.3V" (id 1) (at 323.9389 77.47 90))
+    (in_bom yes) (on_board yes)
+    (property "Reference" "C53" (id 0) (at 324.485 78.105 90))
+    (property "Value" "50μF/6.3V" (id 1) (at 324.485 84.455 90))
     (property "Footprint" "" (id 2) (at 324.485 81.28 0)
       (effects (font (size 1.27 1.27)) hide)
@@
   )
   (symbol (lib_id "Device:C_Polarized_Small") (at 324.485 97.79 90) (unit 1)
-    (in_bom yes) (on_board yes) (fields_autoplaced)
-    (property "Reference" "C55" (id 0) (at 323.9389 91.44 90))
-    (property "Value" "50μF/6.3V" (id 1) (at 323.9389 93.98 90))
+    (in_bom yes) (on_board yes)
+    (property "Reference" "C55" (id 0) (at 324.485 94.615 90))
+    (property "Value" "50μF/6.3V" (id 1) (at 324.485 100.965 90))
     (property "Footprint" "" (id 2) (at 324.485 97.79 0)
       (effects (font (size 1.27 1.27)) hide)
@@
   (symbol (lib_id "Connector:DIN-7") (at 360.934 70.358 180) (unit 1)
     (in_bom yes) (on_board yes) (fields_autoplaced)
-    (property "Reference" "X5" (id 0) (at 360.9339 60.452 0))
-    (property "Value" "DIN-7" (id 1) (at 360.9339 62.992 0))
+    (property "Reference" "X5" (id 0) (at 360.9339 59.69 0))
+    (property "Value" "Video" (id 1) (at 360.9339 62.23 0))
     (property "Footprint" "" (id 2) (at 360.934 70.358 0)
       (effects (font (size 1.27 1.27)) hide)
@@
       (effects (font (size 1.27 1.27)) hide)
     )
-    (property "Value" "" (id 1) (at 91.44 101.6 0))
+    (property "Value" "GND" (id 1) (at 91.44 101.6 0))
     (property "Footprint" "" (id 2) (at 91.44 96.52 0)
       (effects (font (size 1.27 1.27)) hide)
